File: ublox ZED-F9P (Full feature).sch (KiCad schematic (older format))
At the start: 100 parts, among them J1 USB_C_2-LAYER_PADS, J2 CONN_06NO_SILK_FEMALE_PTH, J5 USB_C_2-LAYER_PADS, J6 CONN_06NO_SILK_FEMALE_PTH, U1 LM1117-3.3, U3 ZED-F9P, U4 ZED-F9H

Commit message: Try pushing this repo
Parts:
- B1: partno (none) -> ML414H IV01E
Changed lines of the file:
@@
-3.3V
-Wire Wire Line
-	4300 5900 4300 5800
-Text Label 4300 5900 0    10   ~ 0
 3.3V
 Wire Wire Line
@@
 GND
 Wire Wire Line
-	4300 7300 4300 7200
-Text Label 4300 7300 0    10   ~ 0
-GND
-Wire Wire Line
 	11525 7225 11525 7125
 Text Label 11525 7225 0    10   ~ 0
@@
 ~RESET_P
 Wire Wire Line
-	5900 2000 6000 2000
-Text Label 6000 2000 0    50   ~ 0
-~RESET_P
-Wire Wire Line
 	3125 9675 3025 9675
 Text Label 3025 9675 2    50   ~ 0
-INT_P
-Wire Wire Line
-	5900 2100 6000 2100
-Text Label 6000 2100 0    50   ~ 0
 INT_P
 Wire Wire Line
@@
 Connection ~ 1800 2300
 Wire Wire Line
-	4300 6900 4300 6800
-Wire Wire Line
 	9500 6000 9500 5900
 Wire Wire Line
@@
 	5300 3600 5500 3600
 Wire Wire Line
-	5500 3600 5600 3600
-Wire Wire Line
 	5500 3600 5500 3800
 Wire Wire Line
@@
 Wire Wire Line
 	5300 3500 5500 3500
-Wire Wire Line
-	6100 3600 6000 3600
-Wire Wire Line
-	4300 6300 4300 6400
 $Comp
 L Qwiic_GPS-RTK-SMA_-_ublox_ZED-F9P-eagle-import:GND #GND03
@@
 $EndComp
 $Comp
-L Qwiic_GPS-RTK-SMA_-_ublox_ZED-F9P-eagle-import:ML414H_IV01E_BATTERY B1
-U 1 1 6E38EA6A
-P 1800 6900
-F 0 "B1" H 1800 7070 70  0000 C BNN
-F 1 "6.8MM_COIN_CELL" H 1800 6730 70  0000 C TNN
-F 2 "Qwiic GPS-RTK-SMA - ublox ZED-F9P:ML414H_IV01E" H 1800 6900 50  0001 C CNN
-F 3 "" H 1800 6900 50  0001 C CNN
-	1    1800 6900
-	0    1    1    0
-$EndComp
-$Comp
 L Qwiic_GPS-RTK-SMA_-_ublox_ZED-F9P-eagle-import:GND #GND05
 U 1 1 6CC61BFB
@@
 $EndComp
 $Comp
-L Qwiic_GPS-RTK-SMA_-_ublox_ZED-F9P-eagle-import:33OHM-0603-1_10W-1% R2
-U 1 1 250F4BD6
-P 5700 2200
-F 0 "R2" H 5490 2210 70  0000 C BNN
-F 1 "33" H 5870 2210 70  0000 C BNN
-F 2 "Qwiic GPS-RTK-SMA - ublox ZED-F9P:0603" H 5700 2200 50  0001 C CNN
-F 3 "" H 5700 2200 50  0001 C CNN
-	1    5700 2200
-	1    0    0    -1
-$EndComp
-$Comp
-L Qwiic_GPS-RTK-SMA_-_ublox_ZED-F9P-eagle-import:33OHM-0603-1_10W-1% R4
-U 1 1 83B45A75
-P 5700 2300
-F 0 "R4" H 5490 2310 70  0000 C BNN
-F 1 "33" H 5870 2310 70  0000 C BNN
-F 2 "Qwiic GPS-RTK-SMA - ublox ZED-F9P:0603" H 5700 2300 50  0001 C CNN
-F 3 "" H 5700 2300 50  0001 C CNN
-	1    5700 2300
-	1    0    0    -1
-$EndComp
-$Comp
 L Qwiic_GPS-RTK-SMA_-_ublox_ZED-F9P-eagle-import:3.3V #SUPPLY01
 U 1 1 9BB82FD5
@@
 $EndComp
 $Comp
-L Qwiic_GPS-RTK-SMA_-_ublox_ZED-F9P-eagle-import:1KOHM-0603-1_10W-1% R1
-U 1 1 9D6C0EBA
-P 4300 6600
-F 0 "R1" H 4155 6515 70  0000 C BNN
-F 1 "1k" H 4480 6580 70  0000 C TNN
-F 2 "Qwiic GPS-RTK-SMA - ublox ZED-F9P:0603" H 4300 6600 50  0001 C CNN
-F 3 "" H 4300 6600 50  0001 C CNN
-	1    4300 6600
-	0    -1   -1   0
-$EndComp
-$Comp
-L Qwiic_GPS-RTK-SMA_-_ublox_ZED-F9P-eagle-import:LED-RED0603 LED2
-U 1 1 E7F22A10
-P 4300 7000
-F 0 "LED2" V 4285 6620 70  0000 L BNN
-F 1 "RED" V 4320 6680 70  0000 L TNN
-F 2 "Qwiic GPS-RTK-SMA - ublox ZED-F9P:LED-0603" H 4300 7000 50  0001 C CNN
-F 3 "" H 4300 7000 50  0001 C CNN
-	1    4300 7000
-	1    0    0    -1
-$EndComp
-$Comp
-L Qwiic_GPS-RTK-SMA_-_ublox_ZED-F9P-eagle-import:GND #GND012
-U 1 1 E480151F
-P 4300 7400
-F 0 "#GND012" H 4300 7400 50  0001 C CNN
-F 1 "GND" H 4200 7300 59  0000 L BNN
-F 2 "" H 4300 7400 50  0001 C CNN
-F 3 "" H 4300 7400 50  0001 C CNN
-	1    4300 7400
-	1    0    0    -1
-$EndComp
-$Comp
 L Qwiic_GPS-RTK-SMA_-_ublox_ZED-F9P-eagle-import:0.1UF-0603-25V-5% C5
 U 1 1 6C4A4E38
@@
 $EndComp
 $Comp
-L Qwiic_GPS-RTK-SMA_-_ublox_ZED-F9P-eagle-import:3.3V #P+01
-U 1 1 48DD0DF0
-P 4300 5800
-F 0 "#P+01" H 4300 5800 50  0001 C CNN
-F 1 "3.3V" H 4300 5910 59  0000 C BNN
-F 2 "" H 4300 5800 50  0001 C CNN
-F 3 "" H 4300 5800 50  0001 C CNN
-	1    4300 5800
-	1    0    0    -1
-$EndComp
-$Comp
 L Qwiic_GPS-RTK-SMA_-_ublox_ZED-F9P-eagle-import:1.0UF-0603-16V-10%-X7R C6
 U 1 1 28241604
@@
 $EndComp
 $Comp
-L Qwiic_GPS-RTK-SMA_-_ublox_ZED-F9P-eagle-import:33OHM-0603-1_10W-1% R18
-U 1 1 4E51CAAE
-P 5700 2100
-F 0 "R18" H 5490 2110 70  0000 C BNN
-F 1 "33" H 5870 2110 70  0000 C BNN
-F 2 "Qwiic GPS-RTK-SMA - ublox ZED-F9P:0603" H 5700 2100 50  0001 C CNN
-F 3 "" H 5700 2100 50  0001 C CNN
-	1    5700 2100
-	1    0    0    -1
-$EndComp
-$Comp
-L Qwiic_GPS-RTK-SMA_-_ublox_ZED-F9P-eagle-import:33OHM-0603-1_10W-1% R19
-U 1 1 87DF8B8E
-P 5700 2000
-F 0 "R19" H 5490 2010 70  0000 C BNN
-F 1 "33" H 5870 2010 70  0000 C BNN
-F 2 "Qwiic GPS-RTK-SMA - ublox ZED-F9P:0603" H 5700 2000 50  0001 C CNN
-F 3 "" H 5700 2000 50  0001 C CNN
-	1    5700 2000
-	1    0    0    -1
-$EndComp
-$Comp
 L Qwiic_GPS-RTK-SMA_-_ublox_ZED-F9P-eagle-import:33OHM-0603-1_10W-1% R20
 U 1 1 BFC3FA38
@@
 $EndComp
 $Comp
-L Qwiic_GPS-RTK-SMA_-_ublox_ZED-F9P-eagle-import:JUMPER-SMT_2_NC_TRACE_SILK PPS1
-U 1 1 E4382B22
-P 5800 3600
-F 0 "PPS1" H 5900 3740 70  0000 R TNN
-F 1 "JUMPER-SMT_2_NC_TRACE_SILK" H 5700 3500 70  0000 L TNN
-F 2 "Qwiic GPS-RTK-SMA - ublox ZED-F9P:SMT-JUMPER_2_NC_TRACE_SILK" H 5800 3600 50  0001 C CNN
-F 3 "" H 5800 3600 50  0001 C CNN
-	1    5800 3600
-	-1   0    0    1
-$EndComp
-$Comp
 L Qwiic_GPS-RTK-SMA_-_ublox_ZED-F9P-eagle-import:ANTENNA-GROUNDEDEDGE_SMA E2
 U 1 1 7482DC32
@@
 	1    7500 4000
 	1    0    0    -1
-$EndComp
-$Comp
-L Qwiic_GPS-RTK-SMA_-_ublox_ZED-F9P-eagle-import:JUMPER-SMT_2_NC_TRACE_SILK PWR1
-U 1 1 F8DE81B8
-P 4300 6100
-F 0 "PWR1" H 4220 6170 70  0000 L BNN
-F 1 "JUMPER-SMT_2_NC_TRACE_SILK" H 4200 6000 70  0000 L TNN
-F 2 "Qwiic GPS-RTK-SMA - ublox ZED-F9P:SMT-JUMPER_2_NC_TRACE_SILK" H 4300 6100 50  0001 C CNN
-F 3 "" H 4300 6100 50  0001 C CNN
-	1    4300 6100
-	0    -1   -1   0
 $EndComp
 Text Notes 4800 4300 0    59   ~ 0
@@
 Text Notes 10350 7575 0    50   ~ 0
 10uF tantalum C\n
+$Comp
+L Qwiic_GPS-RTK-SMA_-_ublox_ZED-F9P-eagle-import:33OHM-0603-1_10W-1% R19
+U 1 1 87DF8B8E
+P 5700 2000
+F 0 "R19" H 5490 2010 70  0000 C BNN
+F 1 "33" H 5870 2010 70  0000 C BNN
+F 2 "Qwiic GPS-RTK-SMA - ublox ZED-F9P:0603" H 5700 2000 50  0001 C CNN
+F 3 "" H 5700 2000 50  0001 C CNN
+	1    5700 2000
+	1    0    0    -1
+$EndComp
+$Comp
+L Qwiic_GPS-RTK-SMA_-_ublox_ZED-F9P-eagle-import:33OHM-0603-1_10W-1% R18
+U 1 1 4E51CAAE
+P 5700 2100
+F 0 "R18" H 5490 2110 70  0000 C BNN
+F 1 "33" H 5870 2110 70  0000 C BNN
+F 2 "Qwiic GPS-RTK-SMA - ublox ZED-F9P:0603" H 5700 2100 50  0001 C CNN
+F 3 "" H 5700 2100 50  0001 C CNN
+	1    5700 2100
+	1    0    0    -1
+$EndComp
+$Comp
+L Qwiic_GPS-RTK-SMA_-_ublox_ZED-F9P-eagle-import:33OHM-0603-1_10W-1% R4
+U 1 1 83B45A75
+P 5700 2300
+F 0 "R4" H 5490 2310 70  0000 C BNN
+F 1 "33" H 5870 2310 70  0000 C BNN
+F 2 "Qwiic GPS-RTK-SMA - ublox ZED-F9P:0603" H 5700 2300 50  0001 C CNN
+F 3 "" H 5700 2300 50  0001 C CNN
+	1    5700 2300
+	1    0    0    -1
+$EndComp
+$Comp
+L Qwiic_GPS-RTK-SMA_-_ublox_ZED-F9P-eagle-import:33OHM-0603-1_10W-1% R2
+U 1 1 250F4BD6
+P 5700 2200
+F 0 "R2" H 5490 2210 70  0000 C BNN
+F 1 "33" H 5870 2210 70  0000 C BNN
+F 2 "Qwiic GPS-RTK-SMA - ublox ZED-F9P:0603" H 5700 2200 50  0001 C CNN
+F 3 "" H 5700 2200 50  0001 C CNN
+	1    5700 2200
+	1    0    0    -1
+$EndComp
+Text Label 6000 2100 0    50   ~ 0
+INT_P
+Wire Wire Line
+	5900 2100 6000 2100
+Text Label 6000 2000 0    50   ~ 0
+~RESET_P
+Wire Wire Line
+	5900 2000 6000 2000
+$Comp
+L Qwiic_GPS-RTK-SMA_-_ublox_ZED-F9P-eagle-import:JUMPER-SMT_2_NC_TRACE_SILK PWR1
+U 1 1 F8DE81B8
+P 4300 6100
+F 0 "PWR1" H 4220 6170 70  0000 L BNN
+F 1 "JUMPER-SMT_2_NC_TRACE_SILK" H 4200 6000 70  0000 L TNN
+F 2 "Qwiic GPS-RTK-SMA - ublox ZED-F9P:SMT-JUMPER_2_NC_TRACE_SILK" H 4300 6100 50  0001 C CNN
+F 3 "" H 4300 6100 50  0001 C CNN
+	1    4300 6100
+	0    -1   -1   0
+$EndComp
+$Comp
+L Qwiic_GPS-RTK-SMA_-_ublox_ZED-F9P-eagle-import:3.3V #P+01
+U 1 1 48DD0DF0
+P 4300 5800
+F 0 "#P+01" H 4300 5800 50  0001 C CNN
+F 1 "3.3V" H 4300 5910 59  0000 C BNN
+F 2 "" H 4300 5800 50  0001 C CNN
+F 3 "" H 4300 5800 50  0001 C CNN
+	1    4300 5800
+	1    0    0    -1
+$EndComp
+$Comp
+L Qwiic_GPS-RTK-SMA_-_ublox_ZED-F9P-eagle-import:GND #GND012
+U 1 1 E480151F
+P 4300 7400
+F 0 "#GND012" H 4300 7400 50  0001 C CNN
+F 1 "GND" H 4200 7300 59  0000 L BNN
+F 2 "" H 4300 7400 50  0001 C CNN
+F 3 "" H 4300 7400 50  0001 C CNN
+	1    4300 7400
+	1    0    0    -1
+$EndComp
+$Comp
+L Qwiic_GPS-RTK-SMA_-_ublox_ZED-F9P-eagle-import:LED-RED0603 LED2
+U 1 1 E7F22A10
+P 4300 7000
+F 0 "LED2" V 4285 6620 70  0000 L BNN
+F 1 "RED" V 4320 6680 70  0000 L TNN
+F 2 "Qwiic GPS-RTK-SMA - ublox ZED-F9P:LED-0603" H 4300 7000 50  0001 C CNN
+F 3 "" H 4300 7000 50  0001 C CNN
+	1    4300 7000
+	1    0    0    -1
+$EndComp
+$Comp
+L Qwiic_GPS-RTK-SMA_-_ublox_ZED-F9P-eagle-import:1KOHM-0603-1_10W-1% R1
+U 1 1 9D6C0EBA
+P 4300 6600
+F 0 "R1" H 4155 6515 70  0000 C BNN
+F 1 "1k" H 4480 6580 70  0000 C TNN
+F 2 "Qwiic GPS-RTK-SMA - ublox ZED-F9P:0603" H 4300 6600 50  0001 C CNN
+F 3 "" H 4300 6600 50  0001 C CNN
+	1    4300 6600
+	0    -1   -1   0
+$EndComp
+Wire Wire Line
+	4300 6300 4300 6400
+Wire Wire Line
+	4300 6900 4300 6800
+Text Label 4300 7300 0    10   ~ 0
+GND
+Wire Wire Line
+	4300 7300 4300 7200
+Text Label 4300 5900 0    10   ~ 0
+3.3V
+Wire Wire Line
+	4300 5900 4300 5800
+$Comp
+L Qwiic_GPS-RTK-SMA_-_ublox_ZED-F9P-eagle-import:ML414H_IV01E_BATTERY B1
+U 1 1 6E38EA6A
+P 1800 6900
+F 0 "B1" H 1800 7070 70  0000 C BNN
+F 1 "6.8MM_COIN_CELL" H 1800 6730 70  0000 C TNN
+F 2 "Qwiic GPS-RTK-SMA - ublox ZED-F9P:ML414H_IV01E" H 1800 6900 50  0001 C CNN
+F 3 "" H 1800 6900 50  0001 C CNN
+F 4 "ML414H IV01E" H 1800 6900 50  0001 C CNN "partno"
+	1    1800 6900
+	0    1    1    0
+$EndComp
+Wire Wire Line
+	6100 3600 6000 3600
+Wire Wire Line
+	5500 3600 5600 3600
+$Comp
+L Qwiic_GPS-RTK-SMA_-_ublox_ZED-F9P-eagle-import:JUMPER-SMT_2_NC_TRACE_SILK PPS1
+U 1 1 E4382B22
+P 5800 3600
+F 0 "PPS1" H 5900 3740 70  0000 R TNN
+F 1 "JUMPER-SMT_2_NC_TRACE_SILK" H 5700 3500 70  0000 L TNN
+F 2 "Qwiic GPS-RTK-SMA - ublox ZED-F9P:SMT-JUMPER_2_NC_TRACE_SILK" H 5800 3600 50  0001 C CNN
+F 3 "" H 5800 3600 50  0001 C CNN
+	1    5800 3600
+	-1   0    0    1
+$EndComp
 $EndSCHEMATC

Commit message: Update partno
Parts:
- removed C? (x2): 10uF, symbol Device:CP1
- added C4: 10uF, Qwiic GPS-RTK-SMA - ublox ZED-F9P:0603, symbol Qwiic_GPS-RTK-SMA_-_ublox_ZED-F9P-eagle-import:0.1UF-0603-25V-5%
- C1, C8: partno (none) -> 04023A470KAT2A
- C10, C2, C3, C6, C9: partno (none) -> 0603YC105KAT2A
- C11, C5, C7: partno (none) -> 0603YC104KAT2A
- D10, D3: partno (none) -> HSMG-C120
- D2: partno (none) -> B0520WS-7-F
- D5, D6: value PRTR5V0U2F -> USBLC6-2SC6; footprint Qwiic GPS-RTK-SMA - ublox ZED-F9P:SOT886 -> Package_TO_SOT_SMD:SOT-23-6; partno (none) -> USBLC6-2SC6
- LED1, LED2: partno (none) -> HSMH-C191
- R1, R11, R12, R13, R34, R35, R36, R37, R5: partno (none) -> ERJ-3EKF1001V
- R10, R14, R18, R19, R2, R20, R21, R22, R23, R24, R25, R26, R28, R29, R30, R31, R32, R33, R4, R7, R8, R9: partno (none) -> ERJ-3EKF27R0V
- R15, R27: partno (none) -> ERJ-3EKF1003V
- R16, R17, R3, R6: partno (none) -> ERJ-3EKF5101V
- R38, R39: renamed from R?; partno (none) -> ERJ-3EKF27R0V
- U1: value LM1117-3.3 -> LD1117S33TR; footprint (none) -> Package_TO_SOT_SMD:SOT-223; partno (none) -> LD1117S33TR
- U3: partno (none) -> ZED-F9P-01B
- gave numbers to parts that had none: 12
Connections:
- wire segments 268 -> 265
Other:
- note removed: "10uF tantalum C\n"
- moved on the sheet: U1

Commit message: part no updated
Parts:
- B1: symbol Qwiic_GPS-RTK-SMA_-_ublox_ZED-F9P-eagle-import:ML414H_IV01E_BATTERY -> ublox-ZED-F9P-(Full-feature)-rescue:ML414H_IV01E_BATTERY-Qwiic_GPS-RTK-SMA_-_ublox_ZED-F9P-eagle-import
- C1, C8: symbol Qwiic_GPS-RTK-SMA_-_ublox_ZED-F9P-eagle-import:47PF-0402-25V-5%-X7R -> ublox-ZED-F9P-(Full-feature)-rescue:47PF-0402-25V-5%-X7R-Qwiic_GPS-RTK-SMA_-_ublox_ZED-F9P-eagle-import
- C10, C2, C3, C6, C9: symbol Qwiic_GPS-RTK-SMA_-_ublox_ZED-F9P-eagle-import:1.0UF-0603-16V-10%-X7R -> ublox-ZED-F9P-(Full-feature)-rescue:1.0UF-0603-16V-10%-X7R-Qwiic_GPS-RTK-SMA_-_ublox_ZED-F9P-eagle-import
- C11, C4, C5, C7: symbol Qwiic_GPS-RTK-SMA_-_ublox_ZED-F9P-eagle-import:0.1UF-0603-25V-5% -> ublox-ZED-F9P-(Full-feature)-rescue:0.1UF-0603-25V-5%-Qwiic_GPS-RTK-SMA_-_ublox_ZED-F9P-eagle-import
- D1, D9: symbol Qwiic_GPS-RTK-SMA_-_ublox_ZED-F9P-eagle-import:LED-YELLOW0603 -> ublox-ZED-F9P-(Full-feature)-rescue:LED-YELLOW0603-Qwiic_GPS-RTK-SMA_-_ublox_ZED-F9P-eagle-import; partno (none) -> LY Q396-P1Q2-36
- D10, D3: symbol Qwiic_GPS-RTK-SMA_-_ublox_ZED-F9P-eagle-import:LED-GREEN0603 -> ublox-ZED-F9P-(Full-feature)-rescue:LED-GREEN0603-Qwiic_GPS-RTK-SMA_-_ublox_ZED-F9P-eagle-import
- D11, D4: symbol Qwiic_GPS-RTK-SMA_-_ublox_ZED-F9P-eagle-import:LED-BLUE0603 -> ublox-ZED-F9P-(Full-feature)-rescue:LED-BLUE0603-Qwiic_GPS-RTK-SMA_-_ublox_ZED-F9P-eagle-import; Detailed Description (none) -> Blue 470nm LED Indication - Discrete 3.2V 0603 (1608 Metric); partno (none) -> 150060BS55040
- D2: symbol Qwiic_GPS-RTK-SMA_-_ublox_ZED-F9P-eagle-import:DIODE-SCHOTTKY-PMEG4005EJ -> ublox-ZED-F9P-(Full-feature)-rescue:DIODE-SCHOTTKY-PMEG4005EJ-Qwiic_GPS-RTK-SMA_-_ublox_ZED-F9P-eagle-import
- D5, D6: symbol Qwiic_GPS-RTK-SMA_-_ublox_ZED-F9P-eagle-import:PRTR5V0U2F -> ublox-ZED-F9P-(Full-feature)-rescue:PRTR5V0U2F-Qwiic_GPS-RTK-SMA_-_ublox_ZED-F9P-eagle-import
- D7, D8: partno (none) -> SS34B
- E1, E2, E3, E4: symbol Qwiic_GPS-RTK-SMA_-_ublox_ZED-F9P-eagle-import:ANTENNA-GROUNDEDEDGE_SMA -> ublox-ZED-F9P-(Full-feature)-rescue:ANTENNA-GROUNDEDEDGE_SMA-Qwiic_GPS-RTK-SMA_-_ublox_ZED-F9P-eagle-import; partno (none) -> CON-SMA-EDGE-S
- FB1, FB2: symbol Qwiic_GPS-RTK-SMA_-_ublox_ZED-F9P-eagle-import:FERRITE_BEAD_GNSS -> ublox-ZED-F9P-(Full-feature)-rescue:FERRITE_BEAD_GNSS-Qwiic_GPS-RTK-SMA_-_ublox_ZED-F9P-eagle-import; Detailed Description (none) -> 180 Ohms @ 100MHz 1 Ferrite Bead 0603 (1608 Metric) 2A 50mO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; partno (none) -> BLM15AG100SN1D
- FENCE1, FENCE2, PPS1, PPS2, PPS_LED1, PPS_LED2, PWR1, PWR2, RTK1, RTK2: symbol Qwiic_GPS-RTK-SMA_-_ublox_ZED-F9P-eagle-import:JUMPER-SMT_2_NC_TRACE_SILK -> ublox-ZED-F9P-(Full-feature)-rescue:JUMPER-SMT_2_NC_TRACE_SILK-Qwiic_GPS-RTK-SMA_-_ublox_ZED-F9P-eagle-import; partno (none) -> -
- J1, J5: symbol Qwiic_GPS-RTK-SMA_-_ublox_ZED-F9P-eagle-import:USB_C_2-LAYER_PADS -> ublox-ZED-F9P-(Full-feature)-rescue:USB_C_2-LAYER_PADS-Qwiic_GPS-RTK-SMA_-_ublox_ZED-F9P-eagle-import; partno (none) -> USB-C31-S-RA-EH2.0B-BK-T/R
- J2, J6: symbol Qwiic_GPS-RTK-SMA_-_ublox_ZED-F9P-eagle-import:CONN_06NO_SILK_FEMALE_PTH -> ublox-ZED-F9P-(Full-feature)-rescue:CONN_06NO_SILK_FEMALE_PTH-Qwiic_GPS-RTK-SMA_-_ublox_ZED-F9P-eagle-import
- JP1, JP2, JP3, JP4, JP5, JP6, JP7, JP8: partno (none) -> -
- LED1, LED2: symbol Qwiic_GPS-RTK-SMA_-_ublox_ZED-F9P-eagle-import:LED-RED0603 -> ublox-ZED-F9P-(Full-feature)-rescue:LED-RED0603-Qwiic_GPS-RTK-SMA_-_ublox_ZED-F9P-eagle-import
- R1, R11, R12, R13, R34, R35, R36, R37, R5: symbol Qwiic_GPS-RTK-SMA_-_ublox_ZED-F9P-eagle-import:1KOHM-0603-1_10W-1% -> ublox-ZED-F9P-(Full-feature)-rescue:1KOHM-0603-1_10W-1%-Qwiic_GPS-RTK-SMA_-_ublox_ZED-F9P-eagle-import
- R10, R26, R8, R9: symbol Qwiic_GPS-RTK-SMA_-_ublox_ZED-F9P-eagle-import:27OHM-0603-1_10W-1% -> ublox-ZED-F9P-(Full-feature)-rescue:27OHM-0603-1_10W-1%-Qwiic_GPS-RTK-SMA_-_ublox_ZED-F9P-eagle-import
- R14, R18, R19, R2, R20, R21, R22, R23, R24, R25, R28, R29, R30, R31, R32, R33, R38, R39, R4, R7: symbol Qwiic_GPS-RTK-SMA_-_ublox_ZED-F9P-eagle-import:33OHM-0603-1_10W-1% -> ublox-ZED-F9P-(Full-feature)-rescue:33OHM-0603-1_10W-1%-Qwiic_GPS-RTK-SMA_-_ublox_ZED-F9P-eagle-import
- R15, R27: symbol Qwiic_GPS-RTK-SMA_-_ublox_ZED-F9P-eagle-import:100KOHM-0603-1_10W-1% -> ublox-ZED-F9P-(Full-feature)-rescue:100KOHM-0603-1_10W-1%-Qwiic_GPS-RTK-SMA_-_ublox_ZED-F9P-eagle-import
- R16, R17, R3, R6: symbol Qwiic_GPS-RTK-SMA_-_ublox_ZED-F9P-eagle-import:5.1KOHM5.1KOHM-0603-1_10W-1% -> ublox-ZED-F9P-(Full-feature)-rescue:5.1KOHM5.1KOHM-0603-1_10W-1%-Qwiic_GPS-RTK-SMA_-_ublox_ZED-F9P-eagle-import
- U3: symbol Qwiic_GPS-RTK-SMA_-_ublox_ZED-F9P-eagle-import:ZED-F9P -> ublox-ZED-F9P-(Full-feature)-rescue:ZED-F9P-Qwiic_GPS-RTK-SMA_-_ublox_ZED-F9P-eagle-import
- U4: symbol Qwiic_GPS-RTK-SMA_-_ublox_ZED-F9P-eagle-import:ZED-F9H -> ublox-ZED-F9P-(Full-feature)-rescue:ZED-F9H-Qwiic_GPS-RTK-SMA_-_ublox_ZED-F9P-eagle-import
