File: ublox ZED-F9P (Full feature).sch (KiCad schematic (older format))
At the start: 87 parts, among them J1 USB_C_Receptacle, J2 CONN_06NO_SILK_FEMALE_PTH, J3 USB_C_Receptacle, J4 Molex_PicoBlade, J5 USB_C_2-LAYER_PADS, J6 CONN_06NO_SILK_FEMALE_PTH, J7 JST_GH, U1 LD1117S33TR, U3 ZED-F9P, U4 ZED-F9H

Commit message: changed usb c differential pair
Parts:
- removed J1, J3: USB_C_Receptacle, symbol Connector:USB_C_Receptacle
- removed J5: USB_C_2-LAYER_PADS, Connector_USB:USB_C_Receptacle_GCT_USB4085, symbol ublox-ZED-F9P-(Full-feature)-rescue:USB_C_2-LAYER_PADS-Qwiic_GPS-RTK-SMA_-_ublo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
- removed R6: 5.1k, Qwiic GPS-RTK-SMA - ublox ZED-F9P:0603, symbol ublox-ZED-F9P-(Full-feature)-rescue:5.1KOHM5.1KOHM-0603-1_10W-1%-Qwiic_GPS-RTK-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
- added P1, P2: USB_C_Plug_USB2.0, Connector_USB:USB_C_Receptacle_GCT_USB4085, symbol Connector:USB_C_Receptacle_USB2.0
- added R2: 5.1k, Qwiic GPS-RTK-SMA - ublox ZED-F9P:0603, symbol ublox-ZED-F9P-(Full-feature)-rescue:5.1KOHM5.1KOHM-0603-1_10W-1%-Qwiic_GPS-RTK-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
- added R4, R6: 33, Qwiic GPS-RTK-SMA - ublox ZED-F9P:0603, symbol ublox-ZED-F9P-(Full-feature)-rescue:33OHM-0603-1_10W-1%-Qwiic_GPS-RTK-SMA_-_ubl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
- added TP1, TP2, TP3: TestPoint, TestPoint:TestPoint_Pad_D1.0mm, symbol Connector:TestPoint
Connections:
- net labels added: P_D+, P_D-
- net labels removed: D+_P, D-_P, VBUS
- wire segments 254 -> 253

Commit message: finished routing
Parts:
- added TP4: TestPoint, TestPoint:TestPoint_Pad_D1.0mm, symbol Connector:TestPoint
- C2, C6, C7, C9: footprint Qwiic GPS-RTK-SMA - ublox ZED-F9P:0603 -> Capacitor_SMD:C_0603_1608Metric_Pad1.05x0.95mm_HandSolder
- D12: footprint Diode_SMD:D_SMB_Handsoldering -> Qwiic GPS-RTK-SMA - ublox ZED-F9P:SOD-80; Detailed Description Schottky Barrier Rectifiers Diode 40V/3A -> (none); partno SS34B -> LS4150GS08
- D7, D8: footprint Diode_SMD:D_SMB_Handsoldering -> Qwiic GPS-RTK-SMA - ublox ZED-F9P:SOD-80; partno SS34B -> LS4150GS08
- P1, P2: footprint Connector_USB:USB_C_Receptacle_GCT_USB4085 -> Qwiic GPS-RTK-SMA - ublox ZED-F9P:USB_C_Receptacle_JAE_DX07S016JA1
- R10, R15, R16, R17, R2, R26, R3, R8, R9: footprint Qwiic GPS-RTK-SMA - ublox ZED-F9P:0603 -> Resistor_SMD:R_0603_1608Metric_Pad1.05x0.95mm_HandSolder
Connections:
- net labels added: H_D+, H_D-, _H_D+, _H_D-, _P_D+, _P_D-
- net labels removed: D+_H, D-_H
- wire segments 253 -> 254
Changed lines of the file:
@@
 F 0 "C6" H 9835 6315 70  0000 L BNN
 F 1 "1.0uF" H 9835 6115 70  0000 L BNN
-F 2 "Qwiic GPS-RTK-SMA - ublox ZED-F9P:0603" H 9775 6200 50  0001 C CNN
+F 2 "Capacitor_SMD:C_0603_1608Metric_Pad1.05x0.95mm_HandSolder" H 9775 6200 50  0001 C CNN
 F 3 "" H 9775 6200 50  0001 C CNN
 F 4 "0603YC105KAT2A" H 9775 6200 50  0001 C CNN "partno"
@@
 F 0 "R9" H 2735 3025 70  0000 C BNN
 F 1 "27" H 3085 3010 70  0000 C BNN
-F 2 "Qwiic GPS-RTK-SMA - ublox ZED-F9P:0603" H 2900 3000 50  0001 C CNN
+F 2 "Resistor_SMD:R_0603_1608Metric_Pad1.05x0.95mm_HandSolder" H 2900 3000 50  0001 C CNN
 F 3 "" H 2900 3000 50  0001 C CNN
 F 4 "ERJ-3EKF27R0V" H 2900 3000 50  0001 C CNN "partno"
@@
 F 0 "R10" H 2730 3010 70  0000 C BNN
 F 1 "27" H 3080 3010 70  0000 C BNN
-F 2 "Qwiic GPS-RTK-SMA - ublox ZED-F9P:0603" H 2900 3100 50  0001 C CNN
+F 2 "Resistor_SMD:R_0603_1608Metric_Pad1.05x0.95mm_HandSolder" H 2900 3100 50  0001 C CNN
 F 3 "" H 2900 3100 50  0001 C CNN
 F 4 "ERJ-3EKF27R0V" H 2900 3100 50  0001 C CNN "partno"
@@
 F 0 "R15" H 1925 -1550 70  0000 C BNN
 F 1 "100k" H 3200 3340 70  0000 C TNN
-F 2 "Qwiic GPS-RTK-SMA - ublox ZED-F9P:0603" H 3200 3400 50  0001 C CNN
+F 2 "Resistor_SMD:R_0603_1608Metric_Pad1.05x0.95mm_HandSolder" H 3200 3400 50  0001 C CNN
 F 3 "" H 3200 3400 50  0001 C CNN
 F 4 "ERJ-3EKF1003V" H 3200 3400 50  0001 C CNN "partno"
@@
 F 0 "R16" H 7450 7110 70  0000 C BNN
 F 1 "5.1k" H 7450 6990 70  0000 C TNN
-F 2 "Qwiic GPS-RTK-SMA - ublox ZED-F9P:0603" H 7450 7050 50  0001 C CNN
+F 2 "Resistor_SMD:R_0603_1608Metric_Pad1.05x0.95mm_HandSolder" H 7450 7050 50  0001 C CNN
 F 3 "" H 7450 7050 50  0001 C CNN
 F 4 "ERJ-3EKF5101V" H 7450 7050 50  0001 C CNN "partno"
@@
 F 0 "R17" H 7750 7110 70  0000 C BNN
 F 1 "5.1k" H 7750 6990 70  0000 C TNN
-F 2 "Qwiic GPS-RTK-SMA - ublox ZED-F9P:0603" H 7750 7050 50  0001 C CNN
+F 2 "Resistor_SMD:R_0603_1608Metric_Pad1.05x0.95mm_HandSolder" H 7750 7050 50  0001 C CNN
 F 3 "" H 7750 7050 50  0001 C CNN
 F 4 "ERJ-3EKF5101V" H 7750 7050 50  0001 C CNN "partno"
@@
 	1    5700 3000
 	1    0    0    -1
-$EndComp
-$Comp
-L ublox-ZED-F9P-(Full-feature)-rescue:1.0UF-0603-16V-10%-X7R-Qwiic_GPS-RTK-SMA_-_ublox_ZED-F9P-eagle-import C2
-U 1 1 BFF33B61
-P 3500 3400
-F 0 "C2" V 3470 3280 70  0000 L BNN
-F 1 "1.0uF" V 3590 3130 70  0000 L BNN
-F 2 "Qwiic GPS-RTK-SMA - ublox ZED-F9P:0603" H 3500 3400 50  0001 C CNN
-F 3 "" H 3500 3400 50  0001 C CNN
-F 4 "0603YC105KAT2A" H 3500 3400 50  0001 C CNN "partno"
-	1    3500 3400
-	1    0    0    -1
-$EndComp
-$Comp
-L ublox-ZED-F9P-(Full-feature)-rescue:0.1UF-0603-25V-5%-Qwiic_GPS-RTK-SMA_-_ublox_ZED-F9P-eagle-import C7
-U 1 1 7E3CC750
-P 3800 3300
-F 0 "C7" V 3820 3510 70  0000 R TNN
-F 1 "0.1uF" V 3710 3670 70  0000 R TNN
-F 2 "Qwiic GPS-RTK-SMA - ublox ZED-F9P:0603" H 3800 3300 50  0001 C CNN
-F 3 "" H 3800 3300 50  0001 C CNN
-F 4 "0603YC104KAT2A" H 3800 3300 50  0001 C CNN "partno"
-	1    3800 3300
-	-1   0    0    1
 $EndComp
 $Comp
@@
 F 0 "R8" H 10010 3050 70  0000 C BNN
 F 1 "27" H 10360 3035 70  0000 C BNN
-F 2 "Qwiic GPS-RTK-SMA - ublox ZED-F9P:0603" H 10175 3025 50  0001 C CNN
+F 2 "Resistor_SMD:R_0603_1608Metric_Pad1.05x0.95mm_HandSolder" H 10175 3025 50  0001 C CNN
 F 3 "" H 10175 3025 50  0001 C CNN
 F 4 "ERJ-3EKF27R0V" H 10175 3025 50  0001 C CNN "partno"
@@
 F 0 "R26" H 10005 3035 70  0000 C BNN
 F 1 "27" H 10355 3035 70  0000 C BNN
-F 2 "Qwiic GPS-RTK-SMA - ublox ZED-F9P:0603" H 10175 3125 50  0001 C CNN
+F 2 "Resistor_SMD:R_0603_1608Metric_Pad1.05x0.95mm_HandSolder" H 10175 3125 50  0001 C CNN
 F 3 "" H 10175 3125 50  0001 C CNN
 F 4 "ERJ-3EKF27R0V" H 10175 3125 50  0001 C CNN "partno"
@@
 LQW15ANR12J00D
 Text Label 9875 3125 2    50   ~ 0
-D-_H
+H_D-
 Text Label 9875 3025 2    50   ~ 0
-D+_H
+H_D+
 Wire Wire Line
 	10475 2825 10475 2925
@@
 	9175 8850 9375 8850
 Text Label 9375 8850 0    50   ~ 0
-D+_H
+H_D+
 Wire Wire Line
 	9175 9250 9375 9250
 Text Label 9375 9250 0    50   ~ 0
-D-_H
+H_D-
 $Comp
 L ublox-ZED-F9P-(Full-feature)-rescue:1.0UF-0603-16V-10%-X7R-Qwiic_GPS-RTK-SMA_-_ublox_ZED-F9P-eagle-import C9
@@
 F 0 "C9" H 9835 9065 70  0000 L BNN
 F 1 "1.0uF" H 9835 8865 70  0000 L BNN
-F 2 "Qwiic GPS-RTK-SMA - ublox ZED-F9P:0603" H 9775 8950 50  0001 C CNN
+F 2 "Capacitor_SMD:C_0603_1608Metric_Pad1.05x0.95mm_HandSolder" H 9775 8950 50  0001 C CNN
 F 3 "" H 9775 8950 50  0001 C CNN
 F 4 "0603YC105KAT2A" H 9775 8950 50  0001 C CNN "partno"
@@
 F 0 "D7" H 10075 5693 50  0000 C CNN
 F 1 "D_Small_ALT" H 10075 5784 50  0000 C CNN
-F 2 "Diode_SMD:D_SMB_Handsoldering" V 10075 5900 50  0001 C CNN
-F 3 "https://www.es.co.th/detail.asp?prod=020400218" V 10075 5900 50  0001 C CNN
-F 4 "SS34B" H 10075 5900 50  0001 C CNN "partno"
+F 2 "Qwiic GPS-RTK-SMA - ublox ZED-F9P:SOD-80" V 10075 5900 50  0001 C CNN
+F 3 "https://www.digikey.co.th/product-detail/en/vishay-semiconductor-diodes-division/LS4150GS08/LS4150GS08GICT-ND/4810712" V 10075 5900 50  0001 C CNN
+F 4 "LS4150GS08" H 10075 5900 50  0001 C CNN "partno"
 	1    10075 5900
 	-1   0    0    1
@@
 F 0 "D8" H 10075 8443 50  0000 C CNN
 F 1 "D_Small_ALT" H 10075 8534 50  0000 C CNN
-F 2 "Diode_SMD:D_SMB_Handsoldering" V 10075 8650 50  0001 C CNN
-F 3 "https://www.es.co.th/detail.asp?prod=020400218" V 10075 8650 50  0001 C CNN
-F 4 "SS34B" H 10075 8650 50  0001 C CNN "partno"
+F 2 "Qwiic GPS-RTK-SMA - ublox ZED-F9P:SOD-80" V 10075 8650 50  0001 C CNN
+F 3 "https://www.digikey.co.th/product-detail/en/vishay-semiconductor-diodes-division/LS4150GS08/LS4150GS08GICT-ND/4810712" V 10075 8650 50  0001 C CNN
+F 4 "LS4150GS08" H 10075 8650 50  0001 C CNN "partno"
 	1    10075 8650
 	-1   0    0    1
@@
 F 0 "D12" H 16900 2275 40  0000 R CNN
 F 1 "DIODE" H 16950 2350 40  0000 R CNN
-F 2 "Diode_SMD:D_SMB_Handsoldering" H 16852 2347 60  0001 R CNN
-F 3 "https://www.es.co.th/detail.asp?prod=020400218" H 16746 2347 60  0001 R CNN
-F 4 "SS34B" H 16875 2425 50  0001 C CNN "partno"
-F 5 "Schottky Barrier Rectifiers Diode 40V/3A" H 16875 2425 50  0001 C CNN "Detailed Description"
+F 2 "Qwiic GPS-RTK-SMA - ublox ZED-F9P:SOD-80" H 16852 2347 60  0001 R CNN
+F 3 "https://www.digikey.co.th/product-detail/en/vishay-semiconductor-diodes-division/LS4150GS08/LS4150GS08GICT-ND/4810712" H 16746 2347 60  0001 R CNN
+F 4 "LS4150GS08" H 16875 2425 50  0001 C CNN "partno"
+F 5 "" H 16875 2425 50  0001 C CNN "Detailed Description"
 F 6 "Approved" H 16875 2425 50  0001 C CNN "Approval"
 	1    16875 2425
@@
 F 0 "R2" H 7450 9860 70  0000 C BNN
 F 1 "5.1k" H 7450 9740 70  0000 C TNN
-F 2 "Qwiic GPS-RTK-SMA - ublox ZED-F9P:0603" H 7450 9800 50  0001 C CNN
+F 2 "Resistor_SMD:R_0603_1608Metric_Pad1.05x0.95mm_HandSolder" H 7450 9800 50  0001 C CNN
 F 3 "" H 7450 9800 50  0001 C CNN
 F 4 "ERJ-3EKF5101V" H 7450 9800 50  0001 C CNN "partno"
@@
 F 0 "R3" H 7750 9860 70  0000 C BNN
 F 1 "5.1k" H 7750 9740 70  0000 C TNN
-F 2 "Qwiic GPS-RTK-SMA - ublox ZED-F9P:0603" H 7750 9800 50  0001 C CNN
+F 2 "Resistor_SMD:R_0603_1608Metric_Pad1.05x0.95mm_HandSolder" H 7750 9800 50  0001 C CNN
 F 3 "" H 7750 9800 50  0001 C CNN
 F 4 "ERJ-3EKF5101V" H 7750 9800 50  0001 C CNN "partno"
@@
 F 0 "P2" H 6707 10117 50  0000 C CNN
 F 1 "USB_C_Plug_USB2.0" H 6707 10026 50  0000 C CNN
-F 2 "Connector_USB:USB_C_Receptacle_GCT_USB4085" H 6750 9250 50  0001 C CNN
-F 3 "https://www.usb.org/sites/default/files/documents/usb_type-c.zip" H 6750 9250 50  0001 C CNN
+F 2 "Qwiic GPS-RTK-SMA - ublox ZED-F9P:USB_C_Receptacle_JAE_DX07S016JA1" H 6750 9250 50  0001 C CNN
+F 3 "https://www.mouser.com/ProductDetail/JAE-Electronics/DX07S016JA1R1500?qs=GBLSl2Akirucb2YMMGCxCQ%3D%3D" H 6750 9250 50  0001 C CNN
 	1    6600 9250
 	1    0    0    -1
@@
 F 0 "P1" H 6707 7367 50  0000 C CNN
 F 1 "USB_C_Plug_USB2.0" H 6707 7276 50  0000 C CNN
-F 2 "Connector_USB:USB_C_Receptacle_GCT_USB4085" H 6750 6500 50  0001 C CNN
-F 3 "https://www.usb.org/sites/default/files/documents/usb_type-c.zip" H 6750 6500 50  0001 C CNN
+F 2 "Qwiic GPS-RTK-SMA - ublox ZED-F9P:USB_C_Receptacle_JAE_DX07S016JA1" H 6750 6500 50  0001 C CNN
+F 3 "https://www.mouser.com/ProductDetail/JAE-Electronics/DX07S016JA1R1500?qs=GBLSl2Akirucb2YMMGCxCQ%3D%3D" H 6750 6500 50  0001 C CNN
 	1    6600 6500
 	1    0    0    -1
@@
 	12625 3025 12975 3025
 Wire Wire Line
-	10650 6725 10875 6725
+	10650 6725 10800 6725
 Wire Wire Line
 	8000 6400 8000 6100
@@
 Wire Wire Line
 	8175 6500 8375 6500
+Text Label 8000 6100 0    50   ~ 0
+_P_D-
+Text Label 7950 6600 0    50   ~ 0
+_P_D+
+$Comp
+L Connector:TestPoint TP4
+U 1 1 601ABBBB
+P 10800 6725
+F 0 "TP4" H 10858 6843 50  0000 L CNN
+F 1 "TestPoint" H 10858 6752 50  0000 L CNN
+F 2 "TestPoint:TestPoint_Pad_D1.0mm" H 11000 6725 50  0001 C CNN
+F 3 "~" H 11000 6725 50  0001 C CNN
+	1    10800 6725
+	1    0    0    -1
+$EndComp
+Connection ~ 10800 6725
+Wire Wire Line
+	10800 6725 10875 6725
+Text Label 8175 8850 0    50   ~ 0
+_H_D+
+Text Label 8000 9250 0    50   ~ 0
+_H_D-
+$Comp
+L ublox-ZED-F9P-(Full-feature)-rescue:0.1UF-0603-25V-5%-Qwiic_GPS-RTK-SMA_-_ublox_ZED-F9P-eagle-import C7
+U 1 1 7E3CC750
+P 3800 3300
+F 0 "C7" V 3820 3510 70  0000 R TNN
+F 1 "0.1uF" V 3710 3670 70  0000 R TNN
+F 2 "Capacitor_SMD:C_0603_1608Metric_Pad1.05x0.95mm_HandSolder" H 3800 3300 50  0001 C CNN
+F 3 "" H 3800 3300 50  0001 C CNN
+F 4 "0603YC104KAT2A" H 3800 3300 50  0001 C CNN "partno"
+	1    3800 3300
+	-1   0    0    1
+$EndComp
+$Comp
+L ublox-ZED-F9P-(Full-feature)-rescue:1.0UF-0603-16V-10%-X7R-Qwiic_GPS-RTK-SMA_-_ublox_ZED-F9P-eagle-import C2
+U 1 1 BFF33B61
+P 3500 3400
+F 0 "C2" V 3470 3280 70  0000 L BNN
+F 1 "1.0uF" V 3590 3130 70  0000 L BNN
+F 2 "Capacitor_SMD:C_0603_1608Metric_Pad1.05x0.95mm_HandSolder" H 3500 3400 50  0001 C CNN
+F 3 "" H 3500 3400 50  0001 C CNN
+F 4 "0603YC105KAT2A" H 3500 3400 50  0001 C CNN "partno"
+	1    3500 3400
+	1    0    0    -1
+$EndComp
 $EndSCHEMATC

Commit message: updated new consistent footprint and silkscreen
Parts:
- C10, C11, C3, C4, C5: footprint Qwiic GPS-RTK-SMA - ublox ZED-F9P:0603 -> Capacitor_SMD:C_0603_1608Metric_Pad1.05x0.95mm_HandSolder
- R1, R11, R12, R13, R14, R18, R19, R20, R21, R22, R23, R24, R25, R27, R28, R29, R30, R31, R32, R33, R35, R36, R37, R38, R39, R4, R6, R7: footprint Qwiic GPS-RTK-SMA - ublox ZED-F9P:0603 -> Resistor_SMD:R_0603_1608Metric_Pad1.05x0.95mm_HandSolder

Commit message: finished v1.1
Parts:
- BT1: symbol ublox-ZED-F9P-(Full-feature)-rescue:ML414H_IV01E_BATTERY-Qwiic_GPS-RTK-SMA_-_ublox_ZED-F9P-eagle-import -> ublox-ZED-F9P-(Full-feature)-rescue:ML414H_IV01E_BATTERY-Qwiic_GPS-RTK-SMA_-_ublox_ZED-F9P-eagle-import-ublox-ZED-F9P-(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
- C1, C8: symbol ublox-ZED-F9P-(Full-feature)-rescue:47PF-0402-25V-5%-X7R-Qwiic_GPS-RTK-SMA_-_ublox_ZED-F9P-eagle-import -> ublox-ZED-F9P-(Full-feature)-rescue:47PF-0402-25V-5%-X7R-Qwiic_GPS-RTK-SMA_-_ublox_ZED-F9P-eagle-import-ublox-ZED-F9P-(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
- C10, C2, C3, C6, C9: symbol ublox-ZED-F9P-(Full-feature)-rescue:1.0UF-0603-16V-10%-X7R-Qwiic_GPS-RTK-SMA_-_ublox_ZED-F9P-eagle-import -> ublox-ZED-F9P-(Full-feature)-rescue:1.0UF-0603-16V-10%-X7R-Qwiic_GPS-RTK-SMA_-_ublox_ZED-F9P-eagle-import-ublox-ZED-F9P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
- C11, C4, C5, C7: symbol ublox-ZED-F9P-(Full-feature)-rescue:0.1UF-0603-25V-5%-Qwiic_GPS-RTK-SMA_-_ublox_ZED-F9P-eagle-import -> ublox-ZED-F9P-(Full-feature)-rescue:0.1UF-0603-25V-5%-Qwiic_GPS-RTK-SMA_-_ublox_ZED-F9P-eagle-import-ublox-ZED-F9P-(Ful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
- D2: symbol ublox-ZED-F9P-(Full-feature)-rescue:DIODE-SCHOTTKY-PMEG4005EJ-Qwiic_GPS-RTK-SMA_-_ublox_ZED-F9P-eagle-import -> ublox-ZED-F9P-(Full-feature)-rescue:DIODE-SCHOTTKY-PMEG4005EJ-Qwiic_GPS-RTK-SMA_-_ublox_ZED-F9P-eagle-import-ublox-ZED-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
- D5, D6: symbol ublox-ZED-F9P-(Full-feature)-rescue:PRTR5V0U2F-Qwiic_GPS-RTK-SMA_-_ublox_ZED-F9P-eagle-import -> ublox-ZED-F9P-(Full-feature)-rescue:PRTR5V0U2F-Qwiic_GPS-RTK-SMA_-_ublox_ZED-F9P-eagle-import-ublox-ZED-F9P-(Full-featu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
- E1, E2, E3: symbol ublox-ZED-F9P-(Full-feature)-rescue:ANTENNA-GROUNDEDEDGE_SMA-Qwiic_GPS-RTK-SMA_-_ublox_ZED-F9P-eagle-import -> ublox-ZED-F9P-(Full-feature)-rescue:ANTENNA-GROUNDEDEDGE_SMA-Qwiic_GPS-RTK-SMA_-_ublox_ZED-F9P-eagle-import-ublox-ZED-F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
- FB1, FB2: symbol ublox-ZED-F9P-(Full-feature)-rescue:FERRITE_BEAD_GNSS-Qwiic_GPS-RTK-SMA_-_ublox_ZED-F9P-eagle-import -> ublox-ZED-F9P-(Full-feature)-rescue:FERRITE_BEAD_GNSS-Qwiic_GPS-RTK-SMA_-_ublox_ZED-F9P-eagle-import-ublox-ZED-F9P-(Ful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
- FENCE1, FENCE2, PPS2, PPS_LED1, PPS_LED2, RTK1, RTK2: symbol ublox-ZED-F9P-(Full-feature)-rescue:JUMPER-SMT_2_NC_TRACE_SILK-Qwiic_GPS-RTK-SMA_-_ublox_ZED-F9P-eagle-import -> ublox-ZED-F9P-(Full-feature)-rescue:JUMPER-SMT_2_NC_TRACE_SILK-Qwiic_GPS-RTK-SMA_-_ublox_ZED-F9P-eagle-import-ublox-ZED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
- J2, J6: symbol ublox-ZED-F9P-(Full-feature)-rescue:CONN_06NO_SILK_FEMALE_PTH-Qwiic_GPS-RTK-SMA_-_ublox_ZED-F9P-eagle-import -> ublox-ZED-F9P-(Full-feature)-rescue:CONN_06NO_SILK_FEMALE_PTH-Qwiic_GPS-RTK-SMA_-_ublox_ZED-F9P-eagle-import-ublox-ZED-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
- LED1: symbol ublox-ZED-F9P-(Full-feature)-rescue:LED-RED0603-Qwiic_GPS-RTK-SMA_-_ublox_ZED-F9P-eagle-import -> ublox-ZED-F9P-(Full-feature)-rescue:LED-RED0603-Qwiic_GPS-RTK-SMA_-_ublox_ZED-F9P-eagle-import-ublox-ZED-F9P-(Full-feat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
- LED2, LED5: symbol ublox-ZED-F9P-(Full-feature)-rescue:LED-YELLOW0603-Qwiic_GPS-RTK-SMA_-_ublox_ZED-F9P-eagle-import -> ublox-ZED-F9P-(Full-feature)-rescue:LED-YELLOW0603-Qwiic_GPS-RTK-SMA_-_ublox_ZED-F9P-eagle-import-ublox-ZED-F9P-(Full-f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
- LED3, LED6: symbol ublox-ZED-F9P-(Full-feature)-rescue:LED-GREEN0603-Qwiic_GPS-RTK-SMA_-_ublox_ZED-F9P-eagle-import -> ublox-ZED-F9P-(Full-feature)-rescue:LED-GREEN0603-Qwiic_GPS-RTK-SMA_-_ublox_ZED-F9P-eagle-import-ublox-ZED-F9P-(Full-fe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
- LED4, LED7: symbol ublox-ZED-F9P-(Full-feature)-rescue:LED-BLUE0603-Qwiic_GPS-RTK-SMA_-_ublox_ZED-F9P-eagle-import -> ublox-ZED-F9P-(Full-feature)-rescue:LED-BLUE0603-Qwiic_GPS-RTK-SMA_-_ublox_ZED-F9P-eagle-import-ublox-ZED-F9P-(Full-fea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
- R1, R11, R12, R13, R35, R36, R37, R5: symbol ublox-ZED-F9P-(Full-feature)-rescue:1KOHM-0603-1_10W-1%-Qwiic_GPS-RTK-SMA_-_ublox_ZED-F9P-eagle-import -> ublox-ZED-F9P-(Full-feature)-rescue:1KOHM-0603-1_10W-1%-Qwiic_GPS-RTK-SMA_-_ublox_ZED-F9P-eagle-import-ublox-ZED-F9P-(F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
- R10, R26, R8, R9: symbol ublox-ZED-F9P-(Full-feature)-rescue:27OHM-0603-1_10W-1%-Qwiic_GPS-RTK-SMA_-_ublox_ZED-F9P-eagle-import -> ublox-ZED-F9P-(Full-feature)-rescue:27OHM-0603-1_10W-1%-Qwiic_GPS-RTK-SMA_-_ublox_ZED-F9P-eagle-import-ublox-ZED-F9P-(F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
- R14, R18, R19, R20, R21, R22, R23, R24, R25, R28, R29, R30, R31, R32, R33, R38, R39, R4, R6, R7: symbol ublox-ZED-F9P-(Full-feature)-rescue:33OHM-0603-1_10W-1%-Qwiic_GPS-RTK-SMA_-_ublox_ZED-F9P-eagle-import -> ublox-ZED-F9P-(Full-feature)-rescue:33OHM-0603-1_10W-1%-Qwiic_GPS-RTK-SMA_-_ublox_ZED-F9P-eagle-import-ublox-ZED-F9P-(F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
- R15, R27: symbol ublox-ZED-F9P-(Full-feature)-rescue:100KOHM-0603-1_10W-1%-Qwiic_GPS-RTK-SMA_-_ublox_ZED-F9P-eagle-import -> ublox-ZED-F9P-(Full-feature)-rescue:100KOHM-0603-1_10W-1%-Qwiic_GPS-RTK-SMA_-_ublox_ZED-F9P-eagle-import-ublox-ZED-F9P-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
- R16, R17, R2, R3: symbol ublox-ZED-F9P-(Full-feature)-rescue:5.1KOHM5.1KOHM-0603-1_10W-1%-Qwiic_GPS-RTK-SMA_-_ublox_ZED-F9P-eagle-import -> ublox-ZED-F9P-(Full-feature)-rescue:5.1KOHM5.1KOHM-0603-1_10W-1%-Qwiic_GPS-RTK-SMA_-_ublox_ZED-F9P-eagle-import-ublox-Z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
- U3: symbol ublox-ZED-F9P-(Full-feature)-rescue:ZED-F9P-Qwiic_GPS-RTK-SMA_-_ublox_ZED-F9P-eagle-import -> ublox-ZED-F9P-(Full-feature)-rescue:ZED-F9P-Qwiic_GPS-RTK-SMA_-_ublox_ZED-F9P-eagle-import-ublox-ZED-F9P-(Full-feature)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
- U4: symbol ublox-ZED-F9P-(Full-feature)-rescue:ZED-F9H-Qwiic_GPS-RTK-SMA_-_ublox_ZED-F9P-eagle-import -> ublox-ZED-F9P-(Full-feature)-rescue:ZED-F9H-Qwiic_GPS-RTK-SMA_-_ublox_ZED-F9P-eagle-import-ublox-ZED-F9P-(Full-feature)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

Commit message: genereated output
Parts:
- renumbered D12 to D1
Changed lines of the file:
@@
 EELAYER 30 0
 EELAYER END
-$Descr A2 23386 16535
+$Descr User 19685 12598
 encoding utf-8
 Sheet 1 1
@@
 UART 2 interface\n
 $Comp
-L Device:D_Small_ALT D12
+L Device:D_Small_ALT D1
 U 1 1 5F7085B0
 P 16875 2425
-F 0 "D12" H 16900 2275 40  0000 R CNN
+F 0 "D1" H 16900 2275 40  0000 R CNN
 F 1 "DIODE" H 16950 2350 40  0000 R CNN
 F 2 "Qwiic GPS-RTK-SMA - ublox ZED-F9P:SOD-80" H 16852 2347 60  0001 R CNN

Commit message: rearrange silkscreen H1-H4,P1-P2,J4,J7 remove bottom silkscreen PWR LED resize all footprint references to height0.5,width0.5,thichness0.1 mm Add silkscreen label for pins of J2,J4,J6, J7
Parts:
- D1, D7, D8: symbol Device:D_Small_ALT -> ublox-ZED-F9P-(Full-feature)-rescue:D_Small_ALT-Device
- P1, P2: symbol Connector:USB_C_Receptacle_USB2.0 -> ublox-ZED-F9P-(Full-feature)-rescue:USB_C_Receptacle_USB2.0-Connector
Changed lines of the file:
@@
 $EndComp
 $Comp
-L Device:D_Small_ALT D7
+L ublox-ZED-F9P-(Full-feature)-rescue:D_Small_ALT-Device D7
 U 1 1 5F7307D4
 P 10075 5900
@@
 $EndComp
 $Comp
-L Device:D_Small_ALT D8
+L ublox-ZED-F9P-(Full-feature)-rescue:D_Small_ALT-Device D8
 U 1 1 5F731F06
 P 10075 8650
@@
 UART 2 interface\n
 $Comp
-L Device:D_Small_ALT D1
+L ublox-ZED-F9P-(Full-feature)-rescue:D_Small_ALT-Device D1
 U 1 1 5F7085B0
 P 16875 2425
@@
 	8275 9050 8275 9450
 $Comp
-L Connector:USB_C_Receptacle_USB2.0 P2
+L ublox-ZED-F9P-(Full-feature)-rescue:USB_C_Receptacle_USB2.0-Connector P2
 U 1 1 5F87F742
 P 6600 9250
@@
 Connection ~ 9275 8650
 $Comp
-L Connector:USB_C_Receptacle_USB2.0 P1
+L ublox-ZED-F9P-(Full-feature)-rescue:USB_C_Receptacle_USB2.0-Connector P1
 U 1 1 5F7ACD23
 P 6600 6500
