File: _autosave-ublox ZED-F9P (Full feature).kicad_pcb (KiCad board)
At the start: 4 copper layers, 90 x 50 mm, 92 parts, among them J2 CONN_06NO_SILK_FEMALE_PTH, J4 Molex_PicoBlade, J6 CONN_06NO_SILK_FEMALE_PTH, J7 JST_GH, P1 USB_C_Plug_USB2.0, P2 USB_C_Plug_USB2.0, U1 LD1117S33TR, U3 ZED-F9P, U4 ZED-F9H

Commit message: finished routing
Routing:
- net GND: track 49.1 -> 51.4 mm, vias 266 -> 267
- net Net-(R10-Pad2): track 8.25 -> 9.18 mm
