File: F9R.kicad_pcb (KiCad board)
At the start: 4 copper layers, 90 x 50 mm, 70 parts, among them J1 JST_GH, J2 Molex_PicoBlade, J3 CONN_06NO_SILK_FEMALE_PTH, J4 Conn_01x06, P1 USB_C_Plug_USB2.0, U1 ZED-F9R, U2 DUAL-OPTO_HCPL-073L, U3 LD1117S33TR, U4 UHS_INVERTER_SCHMITT_TRIGGERS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, U5 UHS_INVERTER_SCHMITT_TRIGGERS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

Commit message: finished f9r
Parts:
- added LED4: RED, Qwiic GPS-RTK-SMA - ublox ZED-F9P:LED-0603, F.Cu at (124.7, 71.8)
- added R27: 1k, Resistor_SMD:R_0603_1608Metric_Pad1.05x0.95mm_HandSolder, F.Cu at (128.1, 71.8)
Routing:
- net +3V3: track 90.4 -> 127.2 mm, vias 4 -> 6
- net GND: track 38.2 -> 63.7 mm, vias 21 -> 108
- net Net-(LED4-PadA): track 0.00 -> 1.61 mm

Commit message: added logo
Parts:
- added G***: LOGO, Qwiic GPS-RTK-SMA - ublox ZED-F9P:LOGO_HGR_1cm, B.Cu at (191.9, 92.8)
Other:
- board text added: "PPS"
- board text added: "RTK"
- board text added: "X"
- board text added: "Y"
- board text added: "Z"
- board text added: "fence stat"
- board text removed: "PPS (F9H)"
- board text removed: "RTK (F9H)"
- board text removed: "fence stat (F9H)"
