File: F9R.sch (KiCad schematic (older format))
At the start: 70 parts, among them J1 JST_GH, J2 Molex_PicoBlade, J3 CONN_06NO_SILK_FEMALE_PTH, J4 Conn_01x06, P1 USB_C_Plug_USB2.0, U1 ZED-F9R, U2 DUAL-OPTO_HCPL-073L, U3 LD1117S33TR, U4 UHS_INVERTER_SCHMITT_TRIGGERS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, U5 UHS_INVERTER_SCHMITT_TRIGGERS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

Commit message: finished f9r
Parts:
- added LED4: RED, Qwiic GPS-RTK-SMA - ublox ZED-F9P:LED-0603, symbol ublox-ZED-F9P-(Full-feature)-rescue:LED-RED0603-Qwiic_GPS-RTK-SMA_-_ublox_ZED-F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
- added R27: 1k, Resistor_SMD:R_0603_1608Metric_Pad1.05x0.95mm_HandSolder, symbol ublox-ZED-F9P-(Full-feature)-rescue:1KOHM-0603-1_10W-1%-Qwiic_GPS-RTK-SMA_-_ubl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
- C5: footprint SparkFun_GPS_ZED-F9R_BoB:0402 -> Capacitor_SMD:C_0603_1608Metric_Pad1.05x0.95mm_HandSolder
Connections:
- net +3V3: now also R27.2
- net GND: now also J4.2 (Pin_2), J4.4 (Pin_4), LED4.C; no longer C4.1, U1.G1 (GND), U1.G10 (GND), U1.G11 (GND), U1.G12 (GND), U1.G13 (GND), U1.G14 (GND), U1.G15 (GND), U1.G16 (GND), U1.G17 (GND), U1.G18 (GND), U1.G19 (GND), U1.G2 (GND), U1.G20 (GND), U1.G21 (GND), U1.G22 (GND), U1.G23 (GND), U1.G24 (GND), U1.G25 (GND), U1.G26 (GND), U1.G27 (GND), U1.G28 (GND), U1.G29 (GND), U1.G3 (GND), U1.G30 (GND), U1.G31 (GND), U1.G32 (GND), U1.G33 (GND), U1.G34 (GND), U1.G35 (GND), U1.G36 (GND), U1.G37 (GND), U1.G38 (GND), U1.G39 (GND), U1.G4 (GND), U1.G40 (GND), U1.G41 (GND), U1.G42 (GND), U1.G43 (GND), U1.G44 (GND), U1.G45 (GND), U1.G46 (GND), U1.G47 (GND), U1.G48 (GND), U1.G5 (GND), U1.G6 (GND), U1.G7 (GND), U1.G8 (GND), U1.G9 (GND), U1.P1 (GND), U1.P12 (GND), U1.P14 (GND), U1.P3 (GND), U1.P32 (GND), U1.P37 (GND), U1.P41 (GND), U1.P48 (GND)
- new net: C4.1, U1.G1 (GND), U1.G10 (GND), U1.G11 (GND), U1.G12 (GND), U1.G13 (GND), U1.G14 (GND), U1.G15 (GND), U1.G16 (GND), U1.G17 (GND), U1.G18 (GND), U1.G19 (GND), U1.G2 (GND), U1.G20 (GND), U1.G21 (GND), U1.G22 (GND), U1.G23 (GND), U1.G24 (GND), U1.G25 (GND), U1.G26 (GND), U1.G27 (GND), U1.G28 (GND), U1.G29 (GND), U1.G3 (GND), U1.G30 (GND), U1.G31 (GND), U1.G32 (GND), U1.G33 (GND), U1.G34 (GND), U1.G35 (GND), U1.G36 (GND), U1.G37 (GND), U1.G38 (GND), U1.G39 (GND), U1.G4 (GND), U1.G40 (GND), U1.G41 (GND), U1.G42 (GND), U1.G43 (GND), U1.G44 (GND), U1.G45 (GND), U1.G46 (GND), U1.G47 (GND), U1.G48 (GND), U1.G5 (GND), U1.G6 (GND), U1.G7 (GND), U1.G8 (GND), U1.G9 (GND), U1.P1 (GND), U1.P12 (GND), U1.P14 (GND), U1.P3 (GND), U1.P32 (GND), U1.P37 (GND), U1.P41 (GND), U1.P48 (GND)
- new net: LED4.A, R27.1
- no-connect marks 7 -> 9
